File: Kicad/Data.sch (KiCad schematic (older format))
At the start: 8 parts, among them U11 74HCT574, U12 74HCT574, U13 74HCT574, U14 74HCT574, U15 74HCT541, U16 74HCT541, U23 M27C322-100F1, U24 UM245R

Commit message: Made a slight update to the PCB layout.
Parts:
- U24: footprint Package_DIP:DIP-24_W10.16mm -> Package_DIP:DIP-24_W15.24mm_Socket
Changed lines of the file:
@@
 F 0 "U24" H 9400 1615 50  0000 C CNN
 F 1 "UM245R" H 9400 1524 50  0000 C CNN
-F 2 "Package_DIP:DIP-24_W10.16mm" H 10900 1050 50  0001 L CNN
+F 2 "Package_DIP:DIP-24_W15.24mm_Socket" H 10900 1050 50  0001 L CNN
 F 3 "http://www.ftdichip.com/Support/Documents/DataSheets/Modules/DS_UM245R.pdf" H 10900 950 50  0001 L CNN
 F 4 "UART" H 10900 850 50  0001 L CNN "Description"
@@
 Text Notes 1150 6300 0    50   ~ 0
 Address Bus
-Wire Bus Line
-	3200 700  3200 2250
-Wire Bus Line
-	2750 700  2750 2300
-Wire Bus Line
-	850  700  850  4600
-Wire Bus Line
-	3000 2550 3000 4600
-Wire Bus Line
-	6100 1450 6100 3050
-Wire Bus Line
-	6500 3400 6500 6350
-Wire Bus Line
-	8300 700  8300 5700
 Text Notes 7250 7000 0    50   ~ 0
 The ALU reads from the data bus and the B register. The ALU's output\nis stored in the O register so it can be put back on the data bus.\nBoth the A register and the UART read/write the data bus.\nThe AD buffers allow the hi/low bytes of the address bus to be written to the data bus.
+Wire Bus Line
+	3200 700  3200 2250
+Wire Bus Line
+	2750 700  2750 2300
+Wire Bus Line
+	850  700  850  4600
+Wire Bus Line
+	3000 2550 3000 4600
+Wire Bus Line
+	6100 1450 6100 3050
+Wire Bus Line
+	6500 3400 6500 6350
+Wire Bus Line
+	8300 700  8300 5700
 $EndSCHEMATC
